File: bitaxeNaja.kicad_sch (KiCad schematic)
At the start: 9 parts, among them J1 XT30

Commit message: make the PCB bigger for 70mm heatsink mounting holes
Parts:
- added HS2: Heatsink, bitaxe:70mm-mounting_HTPC, symbol bitaxe:Heatsink
Connections:
- no-connect marks 5 -> 10
Changed lines of the file:
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@@
+	)
+	(no_connect
+		(at 48.26 144.78)
 	)
 	(no_connect
@@
 	)
 	(no_connect
+		(at 48.26 152.4)
+	)
+	(no_connect
+		(at 48.26 149.86)
+	)
+	(no_connect
+		(at 48.26 147.32)
+	)
+	(no_connect
 		(at 48.26 170.18)
 	)
 	(no_connect
 		(at 48.26 162.56)
+	)
+	(no_connect
+		(at 48.26 142.24)
 	)
 	(wire
@@
 			)
 		)
+	)
+	(symbol
+		(lib_id "bitaxe:Heatsink")
+		(at 50.8 139.7 0)
+		(unit 1)
+		(body_style 1)
+		(exclude_from_sim yes)
+		(in_bom no)
+		(on_board yes)
+		(in_pos_files yes)
+		(dnp no)
+		(property "Reference" "HS2"
+			(at 54.61 136.652 0)
+			(show_name no)
+			(do_not_autoplace no)
+			(effects
+				(font
+					(size 1.27 1.27)
+				)
+				(justify left)
+			)
+		)
+		(property "Value" "Heatsink"
+			(at 54.61 139.192 0)
+			(show_name no)
+			(do_not_autoplace no)
+			(effects
+				(font
+					(size 1.27 1.27)
+				)
+				(justify left)
+			)
+		)
+		(property "Footprint" "bitaxe:70mm-mounting_HTPC"
+			(at 51.1048 139.7 0)
+			(hide yes)
+			(show_name no)
+			(do_not_autoplace no)
+			(effects
+				(font
+					(size 1.27 1.27)
+				)
+			)
+		)
+		(property "Datasheet" ""
+			(at 51.1048 139.7 0)
+			(hide yes)
+			(show_name no)
+			(do_not_autoplace no)
+			(effects
+				(font
+					(size 1.27 1.27)
+				)
+			)
+		)
+		(property "Description" "Heatsink"
+			(at 50.8 139.7 0)
+			(hide yes)
+			(show_name no)
+			(do_not_autoplace no)
+			(effects
+				(font
+					(size 1.27 1.27)
+				)
+			)
+		)
+		(property "Manufacturer" ""
+			(at 50.8 139.7 0)
+			(hide yes)
+			(show_name no)
+			(do_not_autoplace no)
+			(effects
+				(font
+					(size 1.27 1.27)
+				)
+			)
+		)
+		(property "Sim.Device" ""
+			(at 50.8 139.7 0)
+			(hide yes)
+			(show_name no)
+			(do_not_autoplace no)
+			(effects
+				(font
+					(size 1.27 1.27)
+				)
+			)
+		)
+		(property "Sim.Pins" ""
+			(at 50.8 139.7 0)
+			(hide yes)
+			(show_name no)
+			(do_not_autoplace no)
+			(effects
+				(font
+					(size 1.27 1.27)
+				)
+			)
+		)
+		(pin "1"
+		)
+		(pin "4"
+		)
+		(pin "5"
+		)
+		(pin "2"
+		)
+		(pin "3"
+		)
+		(instances
+			(project "bitaxeNaja"
+				(path "/61fe8d2c-9301-4ad9-8caf-c47acfa835b0"
+					(reference "HS2")
+					(unit 1)
+				)
+			)
+		)
