File: ASIC.kicad_sch (KiCad schematic)
At the start: 86 parts, among them U10 TLV77308PDBVR, U11 TLV77312PDBVR, U12 TLV77308PDBVR, U14 TLV77312PDBVR, U15 25MHz, U2 SN74AXC4T774, U8 25MHz

Commit message: first pass DFM
Parts:
- added C22, C23: 100nf, Capacitor_SMD:C_0402_1005Metric, symbol Device:C_Small
- added C47, C50: 33pF, Capacitor_SMD:C_0402_1005Metric, symbol Device:C_Small
- U2: footprint bitaxe:BQB0016A-MFG -> Package_SO:TSSOP-16_4.4x5mm_P0.65mm
Connections:
- net GND: now also C22.1, C47.1
- net GND_1: now also C22.2, C23.1, C47.2, C50.1
- net VDD: now also C23.2, C50.2

Commit message: cleaned up kicad trailing whitespace warnings and normalized capacitor units
Parts:
- C22, C23: value 100nf -> 0.1uF
Changed lines of the file:
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@@
 			)
 		)
-		(property "Value" "100nf"
+		(property "Value" "0.1uF"
 			(at 264.922 44.704 0)
 			(show_name no)
@@
 			(at 262.89 43.18 90)
 			(hide yes)
-			(show_name no)
-			(do_not_autoplace no)
-			(effects
-				(font
-					(size 1.27 1.27)
-				)
-			)
-		)
-		(property "Manufacturer" ""
-			(at 262.89 43.18 90)
-			(hide yes)
-			(show_name no)
-			(do_not_autoplace no)
-			(effects
-				(font
-					(size 1.27 1.27)
-				)
-			)
-		)
-		(property "Manufacturer " ""
-			(at 262.89 43.18 0)
 			(show_name no)
 			(do_not_autoplace no)
@@
 			)
 		)
-		(property "Value" "100nf"
+		(property "Value" "0.1uF"
 			(at 263.652 153.924 0)
 			(show_name no)
@@
 			(show_name no)
 			(do_not_autoplace no)
-			(effects
-				(font
-					(size 1.27 1.27)
-				)
-			)
-		)
-		(property "Manufacturer" ""
-			(at 261.62 152.4 90)
-			(hide yes)
-			(show_name no)
-			(do_not_autoplace no)
-			(effects
-				(font
-					(size 1.27 1.27)
-				)
-			)
-		)
-		(property "Manufacturer " ""
-			(at 261.62 152.4 0)
-			(show_name no)
-			(do_not_autoplace no)

Commit message: footprint, BOM cleanup. bypass capacitor spacing cleanup
Parts:
- U2: symbol bitaxe:SN74AVC4T774-BQB -> bitaxe:SN74AXC4T774PWR; DK 296-SN74AXC4T774BQBRCT-ND -> 296-SN74AXC4T774PWRCT-ND; LCSC (none) -> C1849453; PARTNO SN74AXC4T774BQBR -> SN74AXC4T774PWR
Changed lines of the file:
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@@
 	)
 	(symbol
-		(lib_id "bitaxe:SN74AVC4T774-BQB")
+		(lib_id "bitaxe:SN74AXC4T774PWR")
 		(at 77.47 184.15 0)
 		(unit 1)
@@
 		(in_pos_files yes)
 		(dnp no)
-		(fields_autoplaced yes)
 		(property "Reference" "U2"
-			(at 77.47 168.91 0)
+			(at 77.47 169.418 0)
 			(show_name no)
 			(do_not_autoplace no)
@@
 			)
 		)
-		(property "DK" "296-SN74AXC4T774BQBRCT-ND"
+		(property "DK" "296-SN74AXC4T774PWRCT-ND"
 			(at 78.486 210.058 0)
 			(hide yes)
@@
 			)
 		)
-		(property "PARTNO" "SN74AXC4T774BQBR"
-			(at 77.47 184.15 0)
+		(property "PARTNO" "SN74AXC4T774PWR"
+			(at 78.486 203.962 0)
 			(hide yes)
 			(show_name no)
@@
 		(property "Mouser" ""
 			(at 77.47 184.15 0)
+			(hide yes)
+			(show_name no)
+			(do_not_autoplace no)
+			(effects
+				(font
+					(size 1.27 1.27)
+				)
+			)
+		)
+		(property "LCSC" "C1849453"
+			(at 77.216 201.93 0)
 			(hide yes)
 			(show_name no)
@@
 		(pin "8"
 		)
-		(pin "17"
-		)
 		(instances

Commit message: fix all DRC and ERC
Other:
- moved on the sheet: C99, U15
Changed lines of the file:
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@@
 	)
 	(junction
+		(at 199.39 148.59)
+		(diameter 0)
+		(color 0 0 0 0)
+	)
+	(junction
 		(at 224.79 231.14)
 		(diameter 0)
@@
 	)
 	(junction
-		(at 310.642 53.34)
+		(at 311.15 53.34)
 		(diameter 0)
 		(color 0 0 0 0)
@@
 	)
 	(junction
-		(at 330.962 53.34)
+		(at 331.47 53.34)
 		(diameter 0)
 		(color 0 0 0 0)
@@
 	(wire
 		(pts
-			(xy 330.962 53.34) (xy 330.962 62.23)
+			(xy 331.47 53.34) (xy 331.47 62.23)
 		)
 		(stroke
@@
 	(wire
 		(pts
-			(xy 303.53 82.55) (xy 303.53 120.142)
+			(xy 303.53 82.55) (xy 303.53 120.65)
 		)
 		(stroke
@@
 	(wire
 		(pts
-			(xy 337.312 53.34) (xy 330.962 53.34)
+			(xy 337.82 53.34) (xy 331.47 53.34)
 		)
 		(stroke
@@
 	(wire
 		(pts
-			(xy 330.962 62.23) (xy 323.342 62.23)
+			(xy 331.47 62.23) (xy 323.85 62.23)
 		)
 		(stroke
@@
 	(wire
 		(pts
-			(xy 300.99 85.09) (xy 300.99 120.142)
+			(xy 300.99 85.09) (xy 300.99 120.65)
 		)
 		(stroke
@@
 	(wire
 		(pts
-			(xy 295.91 90.17) (xy 295.91 120.142)
+			(xy 295.91 90.17) (xy 295.91 120.65)
 		)
 		(stroke
@@
 	(wire
 		(pts
-			(xy 310.642 53.34) (xy 300.482 53.34)
+			(xy 311.15 53.34) (xy 300.99 53.34)
 		)
 		(stroke
@@
 	(wire
 		(pts
-			(xy 298.45 87.63) (xy 298.45 120.142)
+			(xy 298.45 87.63) (xy 298.45 120.65)
 		)
 		(stroke
@@
 	(wire
 		(pts
-			(xy 312.42 120.142) (xy 312.42 115.57)
+			(xy 312.42 120.65) (xy 312.42 115.57)
 		)
 		(stroke
@@
 	(wire
 		(pts
-			(xy 310.642 62.23) (xy 318.262 62.23)
+			(xy 311.15 62.23) (xy 318.77 62.23)
 		)
 		(stroke
@@
 	(wire
 		(pts
-			(xy 310.642 53.34) (xy 310.642 62.23)
+			(xy 311.15 53.34) (xy 311.15 62.23)
 		)
 		(stroke
@@
 	(wire
 		(pts
-			(xy 328.422 53.34) (xy 330.962 53.34)
+			(xy 328.93 53.34) (xy 331.47 53.34)
 		)
 		(stroke
@@
 	(wire
 		(pts
-			(xy 313.182 53.34) (xy 310.642 53.34)
+			(xy 313.69 53.34) (xy 311.15 53.34)
 		)
 		(stroke
@@
 	(wire
 		(pts
-			(xy 306.07 80.01) (xy 306.07 120.142)
+			(xy 306.07 80.01) (xy 306.07 120.65)
 		)
 		(stroke
@@
 	(wire
 		(pts
-			(xy 290.83 120.142) (xy 290.83 115.57)
+			(xy 290.83 120.65) (xy 290.83 115.57)
 		)
 		(stroke
@@
 	(wire
 		(pts
-			(xy 313.182 50.8) (xy 294.64 50.8)
+			(xy 313.69 50.8) (xy 294.64 50.8)
 		)
 		(stroke
@@
 	(wire
 		(pts
-			(xy 337.312 50.8) (xy 328.422 50.8)
+			(xy 337.82 50.8) (xy 328.93 50.8)
 		)
 		(stroke
@@
 	)
 	(label "1V2_1"
-		(at 337.312 50.8 180)
+		(at 337.82 50.8 180)
 		(effects
 			(font
@@
 	)
 	(label "GND_1"
-		(at 337.312 53.34 180)
+		(at 337.82 53.34 180)
 		(effects
 			(font
@@
 	)
 	(label "1V2_1"
-		(at 300.482 53.34 0)
+		(at 300.99 53.34 0)
 		(effects
 			(font
@@
 	)
 	(symbol
+		(lib_id "power:PWR_FLAG")
+		(at 199.39 148.59 0)
+		(unit 1)
+		(body_style 1)
+		(exclude_from_sim no)
+		(in_bom yes)
+		(on_board yes)
+		(in_pos_files yes)
+		(dnp no)
+		(fields_autoplaced yes)
+		(property "Reference" "#FLG01"
+			(at 199.39 146.685 0)
+			(hide yes)
+			(show_name no)
+			(do_not_autoplace no)
+			(effects
+				(font
+					(size 1.27 1.27)
+				)
+			)
+		)
+		(property "Value" "GND_1"
+			(at 199.39 143.51 0)
+			(show_name no)
+			(do_not_autoplace no)
+			(effects
+				(font
+					(size 1.27 1.27)
+				)
+			)
+		)
+		(property "Footprint" ""
+			(at 199.39 148.59 0)
+			(hide yes)
+			(show_name no)
+			(do_not_autoplace no)
+			(effects
+				(font
+					(size 1.27 1.27)
+				)
+			)
+		)
+		(property "Datasheet" ""
+			(at 199.39 148.59 0)
+			(hide yes)
+			(show_name no)
+			(do_not_autoplace no)
+			(effects
+				(font
+					(size 1.27 1.27)
+				)
+			)
+		)
+		(property "Description" "Special symbol for telling ERC where power comes from"
+			(at 199.39 148.59 0)
+			(hide yes)
+			(show_name no)
+			(do_not_autoplace no)
+			(effects
+				(font
+					(size 1.27 1.27)
+				)
+			)
+		)
+		(pin "1"
+		)
+		(instances
+			(project "bitaxeNaja"
+				(path "/61fe8d2c-9301-4ad9-8caf-c47acfa835b0/5053a6d5-ae8d-4ae0-9f6e-0d65e80da719"
+					(reference "#FLG01")
+					(unit 1)
+				)
+			)
+		)
+	)
+	(symbol
 		(lib_id "Regulator_Linear:TLV73312PDBV")
 		(at 369.57 73.66 0)
@@
 	(symbol
 		(lib_id "bitaxe:oscillator")
-		(at 320.802 52.07 0)
+		(at 321.31 52.07 0)
 		(mirror y)
 		(unit 1)
@@
 		(dnp no)
 		(property "Reference" "U15"
-			(at 320.802 46.482 0)
+			(at 321.31 46.482 0)
 			(show_name no)
 			(do_not_autoplace no)
@@
 		)
 		(property "Value" "25MHz"
-			(at 320.294 57.404 0)
+			(at 320.802 57.404 0)
 			(show_name no)
 			(do_not_autoplace no)
@@
 		)
 		(property "Footprint" "bitaxe:SMD3225-4P"
-			(at 322.072 53.34 0)
+			(at 322.58 53.34 0)
 			(hide yes)
 			(show_name no)
@@
 		)
 		(property "Datasheet" ""
-			(at 322.072 53.34 0)
+			(at 322.58 53.34 0)
 			(hide yes)
 			(show_name no)
@@
 		)
 		(property "Description" ""
-			(at 320.802 52.07 0)
+			(at 321.31 52.07 0)
 			(hide yes)
 			(show_name no)
@@
 		)
 		(property "DK" "5852-SX3M25.000E20F30THNTR-ND"
-			(at 320.802 52.07 0)
+			(at 321.31 52.07 0)
 			(hide yes)
 			(show_name no)
@@
 		)
 		(property "LCSC" "C5137262"
-			(at 320.802 52.07 0)
+			(at 321.31 52.07 0)
 			(hide yes)
 			(show_name no)
@@
 		)
 		(property "PARTNO" "SX3M25.000E20F30THN"
-			(at 320.802 52.07 0)
+			(at 321.31 52.07 0)
 			(hide yes)
 			(show_name no)
@@
 		)
 		(property "Mouser" ""
-			(at 320.802 52.07 0)
+			(at 321.31 52.07 0)
 			(hide yes)
 			(show_name no)
@@
 	(symbol
 		(lib_id "Device:C_Small")
-		(at 320.802 62.23 90)
+		(at 321.31 62.23 90)
 		(mirror x)
 		(unit 1)
@@
 		(dnp no)
 		(property "Reference" "C99"
-			(at 318.77 65.278 90)
+			(at 319.278 65.278 90)
 			(show_name no)
 			(do_not_autoplace no)
@@
 		)
 		(property "Value" "0.1uF"
-			(at 318.008 67.056 90)
+			(at 318.516 67.056 90)
 			(show_name no)
 			(do_not_autoplace no)
@@
 		)
 		(property "Footprint" "Capacitor_SMD:C_0402_1005Metric"
-			(at 320.802 62.23 0)
+			(at 321.31 62.23 0)
 			(hide yes)
 			(show_name no)
@@
 		)
 		(property "Datasheet" "https://datasheets.kyocera-avx.com/KGM_X7R.pdf"
-			(at 320.802 62.23 0)
+			(at 321.31 62.23 0)
 			(hide yes)
 			(show_name no)
@@
 		)
 		(property "Description" "Unpolarized capacitor, small symbol"
-			(at 320.802 62.23 0)
+			(at 321.31 62.23 0)
 			(hide yes)
 			(show_name no)
@@
 		)
 		(property "PARTNO" "KGM05AR71C104KH"
-			(at 320.802 62.23 0)
+			(at 321.31 62.23 0)
 			(hide yes)
 			(show_name no)
@@
 		)
 		(property "DK" "478-KGM05AR71C104KHCT-ND"
-			(at 320.802 62.23 0)
+			(at 321.31 62.23 0)
 			(hide yes)
 			(show_name no)
@@
 		)
 		(property "Mouser" ""
-			(at 320.802 62.23 90)
+			(at 321.31 62.23 90)
 			(hide yes)
 			(show_name no)
@@
 	)
 	(sheet
-		(at 288.544 120.142)
-		(size 25.908 23.368)
+		(at 288.29 120.65)
+		(size 26.162 22.86)
 		(exclude_from_sim no)
 		(in_bom yes)
@@
 		)
 		(property "Sheetname" "Level Shifter"
-			(at 287.8324 143.51 90)
+			(at 287.5784 144.018 90)
 			(show_name no)
 			(do_not_autoplace no)
@@
 		)
 		(property "Sheetfile" "level_shifter.kicad_sch"
-			(at 315.214 145.288 90)
+			(at 314.96 145.796 90)
 			(show_name no)
 			(do_not_autoplace no)
@@
 		)
 		(pin "BO" input
-			(at 306.07 120.142 90)
+			(at 306.07 120.65 90)
 			(effects
 				(font
@@
 		)
 		(pin "CO" input
-			(at 298.45 120.142 90)
+			(at 298.45 120.65 90)
 			(effects
 				(font
@@
 		)
 		(pin "GND_HI" input
-			(at 312.42 120.142 90)
+			(at 312.42 120.65 90)
 			(effects
 				(font
@@
 		)
 		(pin "NRSTO" input
-			(at 295.91 120.142 90)
+			(at 295.91 120.65 90)
 			(effects
 				(font
@@
 		)
 		(pin "RI" input
-			(at 300.99 120.142 90)
+			(at 300.99 120.65 90)
 			(effects
 				(font
@@
 		)
 		(pin "VDD_HI" input
-			(at 290.83 120.142 90)
+			(at 290.83 120.65 90)
 			(effects
 				(font
@@
 		)
 		(pin "CLKO" input
-			(at 303.53 120.142 90)
+			(at 303.53 120.65 90)
 			(effects
 				(font

Commit message: moved the 3V3 level shifter down out of the main GND power plane. BOM cleanup
Parts:
- C22, C23: DK (none) -> 490-10700-1-ND; LCSC (none) -> C77020; PARTNO GRM188R61E106KA73D -> GRM155R71H104KE14D

Commit message: bumped version to 1201xx. added fixes for #3
Parts:
- added R74, R76: 33, Resistor_SMD:R_0402_1005Metric, symbol Device:R_US
- C99, U15: now not fitted
Connections:
- net Level Shifter/CI: now also R74.2; no longer A1.25 (CO)
- net Level Shifter/RI: now also R76.2; no longer A2.24 (RO)
- new net: A1.25 (CO), R74.1
- new net: A2.24 (RO), R76.1
Changed lines of the file:
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@@
 		(title "bitaxeNaja")
 		(date "2026-06-18")
-		(rev "1201x")
+		(rev "1201xx")
 		(company "bitaxeorg")
 		(comment 1 "OHL v2")
@@
 	(wire
 		(pts
+			(xy 232.41 191.77) (xy 271.78 191.77)
+		)
+		(stroke
+			(width 0)
+			(type default)
+		)
+	)
+	(wire
+		(pts
 			(xy 176.53 224.79) (xy 176.53 231.14)
 		)
@@
 	(wire
 		(pts
-			(xy 214.63 191.77) (xy 271.78 191.77)
+			(xy 214.63 191.77) (xy 224.79 191.77)
 		)
 		(stroke
@@
 	(wire
 		(pts
+			(xy 228.6 85.09) (xy 271.78 85.09)
+		)
+		(stroke
+			(width 0)
+			(type default)
+		)
+	)
+	(wire
+		(pts
 			(xy 271.78 90.17) (xy 295.91 90.17)
 		)
@@
 	(wire
 		(pts
-			(xy 214.63 85.09) (xy 271.78 85.09)
+			(xy 214.63 85.09) (xy 220.98 85.09)
 		)
 		(stroke
@@
 	)
 	(symbol
+		(lib_id "Device:R_US")
+		(at 228.6 191.77 90)
+		(unit 1)
+		(body_style 1)
+		(exclude_from_sim no)
+		(in_bom yes)
+		(on_board yes)
+		(in_pos_files yes)
+		(dnp no)
+		(property "Reference" "R74"
+			(at 224.028 190.754 90)
+			(show_name no)
+			(do_not_autoplace no)
+			(effects
+				(font
+					(size 1.27 1.27)
+				)
+			)
+		)
+		(property "Value" "33"
+			(at 232.664 190.754 90)
+			(show_name no)
+			(do_not_autoplace no)
+			(effects
+				(font
+					(size 1.27 1.27)
+				)
+			)
+		)
+		(property "Footprint" "Resistor_SMD:R_0402_1005Metric"
+			(at 228.854 190.754 90)
+			(hide yes)
+			(show_name no)
+			(do_not_autoplace no)
+			(effects
+				(font
+					(size 1.27 1.27)
+				)
+			)
+		)
+		(property "Datasheet" ""
+			(at 228.6 191.77 0)
+			(hide yes)
+			(show_name no)
+			(do_not_autoplace no)
+			(effects
+				(font
+					(size 1.27 1.27)
+				)
+			)
+		)
+		(property "Description" "Resistor, US symbol"
+			(at 228.6 191.77 0)
+			(hide yes)
+			(show_name no)
+			(do_not_autoplace no)
+			(effects
+				(font
+					(size 1.27 1.27)
+				)
+			)
+		)
+		(property "PARTNO" ""
+			(at 228.6 191.77 90)
+			(hide yes)
+			(show_name no)
+			(do_not_autoplace no)
+			(effects
+				(font
+					(size 1.27 1.27)
+				)
+			)
+		)
+		(property "Mouser" ""
+			(at 228.6 191.77 90)
+			(hide yes)
+			(show_name no)
+			(do_not_autoplace no)
+			(effects
+				(font
+					(size 1.27 1.27)
+				)
+			)
+		)
+		(pin "1"
+		)
+		(pin "2"
+		)
+		(instances
+			(project "bitaxeNaja"
+				(path "/61fe8d2c-9301-4ad9-8caf-c47acfa835b0/5053a6d5-ae8d-4ae0-9f6e-0d65e80da719"
+					(reference "R74")
+					(unit 1)
+				)
+			)
+		)
+	)
+	(symbol
 		(lib_id "Device:C_Small")
 		(at 354.33 102.87 180)
@@
 		(on_board yes)
 		(in_pos_files yes)
-		(dnp no)
+		(dnp yes)
 		(property "Reference" "U15"
 			(at 321.31 46.482 0)
@@
 	)
 	(symbol
+		(lib_id "Device:R_US")
+		(at 224.79 85.09 90)
+		(unit 1)
+		(body_style 1)
+		(exclude_from_sim no)
+		(in_bom yes)
+		(on_board yes)
+		(in_pos_files yes)
+		(dnp no)
+		(property "Reference" "R76"
+			(at 220.218 84.074 90)
+			(show_name no)
+			(do_not_autoplace no)
+			(effects
+				(font
+					(size 1.27 1.27)
+				)
+			)
+		)
+		(property "Value" "33"
+			(at 228.854 84.074 90)
+			(show_name no)
+			(do_not_autoplace no)
+			(effects
+				(font
+					(size 1.27 1.27)
+				)
+			)
+		)
+		(property "Footprint" "Resistor_SMD:R_0402_1005Metric"
+			(at 225.044 84.074 90)
+			(hide yes)
+			(show_name no)
+			(do_not_autoplace no)
+			(effects
+				(font
+					(size 1.27 1.27)
+				)
+			)
+		)
+		(property "Datasheet" ""
+			(at 224.79 85.09 0)
+			(hide yes)
+			(show_name no)
+			(do_not_autoplace no)
+			(effects
+				(font
+					(size 1.27 1.27)
+				)
+			)
+		)
+		(property "Description" "Resistor, US symbol"
+			(at 224.79 85.09 0)
+			(hide yes)
+			(show_name no)
+			(do_not_autoplace no)
+			(effects
+				(font
+					(size 1.27 1.27)
+				)
+			)
+		)
+		(property "PARTNO" ""
+			(at 224.79 85.09 90)
+			(hide yes)
+			(show_name no)
+			(do_not_autoplace no)
+			(effects
+				(font
+					(size 1.27 1.27)
+				)
+			)
+		)
+		(property "Mouser" ""
+			(at 224.79 85.09 90)
+			(hide yes)
+			(show_name no)
+			(do_not_autoplace no)
+			(effects
+				(font
+					(size 1.27 1.27)
+				)
+			)
+		)
+		(pin "1"
+		)
+		(pin "2"
+		)
+		(instances
+			(project "bitaxeNaja"
+				(path "/61fe8d2c-9301-4ad9-8caf-c47acfa835b0/5053a6d5-ae8d-4ae0-9f6e-0d65e80da719"
+					(reference "R76")
+					(unit 1)
+				)
+			)
+		)
+	)
+	(symbol
 		(lib_id "Device:C_Small")
 		(at 170.18 113.03 0)
@@
 		(on_board yes)
 		(in_pos_files yes)
-		(dnp no)
+		(dnp yes)
 		(property "Reference" "C99"
 			(at 319.278 65.278 90)
