File: level_shifter.kicad_sch (KiCad schematic)
At the start: 21 parts, among them U17 TLV3544

Commit message: rough parts placement.
Connections:
- net -VDD2 renamed GND_LO
- net GND2 renamed GND_HI
- net VDD2 renamed VDD_HI
Other:
- company: (none) -> bitaxeorg
- title: (none) -> bitaxeNaja
- moved on the sheet: R72

Commit message: AI BOM updates
Parts:
- C207: LCSC (none) -> C2177690
- R56, R57, R59, R60, R62, R63, R65, R66: LCSC (none) -> C25744

Commit message: fix all DRC and ERC
Changed lines of the file:
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@@
 		)
 	)
-	(label "NRSTI2"
+	(label "NRSTO"
 		(at 168.91 93.98 180)
 		(effects
@@
 		)
 	)
-	(label "RO2"
+	(label "RI"
 		(at 109.22 161.29 0)
 		(effects
@@
 		)
 	)
-	(label "BI2"
+	(label "BO"
 		(at 166.37 123.19 180)
 		(effects
@@
 		)
 	)
-	(label "CI2"
+	(label "CO"
 		(at 166.37 63.5 180)
 		(effects

Commit message: bumped version to 1201xx. added fixes for #3
Parts:
- added C101: 0.01uF, Capacitor_SMD:C_0402_1005Metric, symbol Device:C_Small
- R67: value 0 -> 33; PARTNO RC0402JR-070RL -> (none); now fitted
Connections:
- net CLKO: now also C101.2; no longer R67.2
- new net: C101.1, R67.2
Other:
- note added: "clock domain passthrough."
- note removed: "clock domain passthrough. Ideally this works"
Changed lines of the file:
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@@
 		(title "bitaxeNaja")
 		(date "2026-06-18")
-		(rev "1201x")
+		(rev "1201xx")
 		(company "bitaxeorg")
 		(comment 1 "OHL v2")
@@
 		)
 	)
-	(text "clock domain passthrough. Ideally this works"
+	(text "clock domain passthrough."
 		(exclude_from_sim no)
-		(at 141.224 41.656 0)
+		(at 139.954 31.242 0)
 		(effects
 			(font
@@
 	(wire
 		(pts
+			(xy 152.4 38.1) (xy 172.72 38.1)
+		)
+		(stroke
+			(width 0)
+			(type default)
+		)
+	)
+	(wire
+		(pts
 			(xy 130.81 71.12) (xy 130.81 66.04)
 		)
@@
 	(wire
 		(pts
-			(xy 109.22 38.1) (xy 137.16 38.1)
+			(xy 109.22 38.1) (xy 125.73 38.1)
 		)
 		(stroke
@@
 	(wire
 		(pts
-			(xy 144.78 38.1) (xy 172.72 38.1)
-		)
-		(stroke
-			(width 0)
-			(type default)
-		)
-	)
-	(wire
-		(pts
 			(xy 130.81 49.53) (xy 130.81 60.96)
 		)
@@
 		(pts
 			(xy 130.81 139.7) (xy 142.24 139.7)
+		)
+		(stroke
+			(width 0)
+			(type default)
+		)
+	)
+	(wire
+		(pts
+			(xy 133.35 38.1) (xy 147.32 38.1)
 		)
 		(stroke
@@
 	)
 	(symbol
+		(lib_id "Device:C_Small")
+		(at 149.86 38.1 90)
+		(mirror x)
+		(unit 1)
+		(body_style 1)
+		(exclude_from_sim no)
+		(in_bom yes)
+		(on_board yes)
+		(in_pos_files yes)
+		(dnp no)
+		(property "Reference" "C101"
+			(at 147.574 35.052 90)
+			(show_name no)
+			(do_not_autoplace no)
+			(effects
+				(font
+					(size 1.27 1.27)
+				)
+				(justify right)
+			)
+		)
+		(property "Value" "0.01uF"
+			(at 147.574 41.148 90)
+			(show_name no)
+			(do_not_autoplace no)
+			(effects
+				(font
+					(size 1.27 1.27)
+				)
+				(justify right)
+			)
+		)
+		(property "Footprint" "Capacitor_SMD:C_0402_1005Metric"
+			(at 149.86 38.1 0)
+			(hide yes)
+			(show_name no)
+			(do_not_autoplace no)
+			(effects
+				(font
+					(size 1.27 1.27)
+				)
+			)
+		)
+		(property "Datasheet" "https://datasheets.kyocera-avx.com/KGM_X7R.pdf"
+			(at 149.86 38.1 0)
+			(hide yes)
+			(show_name no)
+			(do_not_autoplace no)
+			(effects
+				(font
+					(size 1.27 1.27)
+				)
+			)
+		)
+		(property "Description" "Unpolarized capacitor, small symbol"
+			(at 149.86 38.1 0)
+			(hide yes)
+			(show_name no)
+			(do_not_autoplace no)
+			(effects
+				(font
+					(size 1.27 1.27)
+				)
+			)
+		)
+		(property "PARTNO" ""
+			(at 149.86 38.1 0)
+			(hide yes)
+			(show_name no)
+			(do_not_autoplace no)
+			(effects
+				(font
+					(size 1.27 1.27)
+				)
+			)
+		)
+		(property "DK" ""
+			(at 149.86 38.1 0)
+			(hide yes)
+			(show_name no)
+			(do_not_autoplace no)
+			(effects
+				(font
+					(size 1.27 1.27)
+				)
+			)
+		)
+		(property "Mouser" ""
+			(at 149.86 38.1 90)
+			(hide yes)
+			(show_name no)
+			(do_not_autoplace no)
+			(effects
+				(font
+					(size 1.27 1.27)
+				)
+			)
+		)
+		(pin "1"
+		)
+		(pin "2"
+		)
+		(instances
+			(project "bitaxeNaja"
+				(path "/61fe8d2c-9301-4ad9-8caf-c47acfa835b0/5053a6d5-ae8d-4ae0-9f6e-0d65e80da719/e54a6d2e-c74f-49ed-b74b-fa12427eb615"
+					(reference "C101")
+					(unit 1)
+				)
+			)
+		)
+	)
+	(symbol
 		(lib_id "Device:R_US")
 		(at 146.05 49.53 270)
@@
 	(symbol
 		(lib_id "Device:R_US")
-		(at 140.97 38.1 90)
+		(at 129.54 38.1 90)
 		(unit 1)
 		(body_style 1)
@@
 		(on_board yes)
 		(in_pos_files yes)
-		(dnp yes)
-		(fields_autoplaced yes)
+		(dnp no)
 		(property "Reference" "R67"
-			(at 140.97 31.75 90)
-			(show_name no)
-			(do_not_autoplace no)
-			(effects
-				(font
-					(size 1.27 1.27)
-				)
-			)
-		)
-		(property "Value" "0"
-			(at 140.97 34.29 90)
+			(at 129.54 35.306 90)
+			(show_name no)
+			(do_not_autoplace no)
+			(effects
+				(font
+					(size 1.27 1.27)
+				)
+			)
+		)
+		(property "Value" "33"
+			(at 129.794 41.148 90)
 			(show_name no)
 			(do_not_autoplace no)
@@
 		)
 		(property "Footprint" "Resistor_SMD:R_0402_1005Metric"
-			(at 141.224 37.084 90)
+			(at 129.794 37.084 90)
 			(hide yes)
 			(show_name no)
@@
 		)
 		(property "Datasheet" ""
-			(at 140.97 38.1 0)
+			(at 129.54 38.1 0)
 			(hide yes)
 			(show_name no)
@@
 		)
 		(property "Description" "Resistor, US symbol"
-			(at 140.97 38.1 0)
-			(hide yes)
-			(show_name no)
-			(do_not_autoplace no)
-			(effects
-				(font
-					(size 1.27 1.27)
-				)
-			)
-		)
-		(property "PARTNO" "RC0402JR-070RL"
-			(at 140.97 38.1 90)
+			(at 129.54 38.1 0)
+			(hide yes)
+			(show_name no)
+			(do_not_autoplace no)
+			(effects
+				(font
+					(size 1.27 1.27)
+				)
+			)
+		)
+		(property "PARTNO" ""
+			(at 129.54 38.1 90)
 			(hide yes)
 			(show_name no)
@@
 		)
 		(property "Mouser" ""
-			(at 140.97 38.1 90)
-			(hide yes)
-			(show_name no)
+			(at 129.54 38.1 90)
+			(hide yes)
+			(show_name no)
